File: PCB/comp pcb1.kicad_pcb (KiCad board)
At the start: 2 copper layers, 46 x 45.5 mm, 35 parts, among them SW1 SW_Push, SW2 SW_Push, U1 STM32F401RETx, U2 regulartor, Y1 8MHz 8MHz

Commit message: Add files via upload
Routing:
- net GND: track 189.1 -> 169.2 mm
- net /Vreg: track 180.4 -> 179.4 mm
